File: FinalTeensyBreakoutBoard/FinalTeensyBreakoutBoard.kicad_pcb (KiCad board)
At the start: 2 copper layers, 38 parts, among them J1 POWER, J2 MC1, J3 MC2, J4 MC3, J5 CurrSB, J6 UWB1, J7 UWBchip, U1 Teensy4.1, U2 MAX3284E, U3 MAX3284E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

Commit message: finished layout
Parts:
- removed 3.3V1, GND1: Conn_01x03_Male, teensy:3pinJST
- added REF**: MountingHole_3.7mm_Pad, MountingHole:MountingHole_3.7mm_Pad, F.Cu at (172.7, 147.3)
- added REF**: MountingHole_3.7mm_Pad, MountingHole:MountingHole_3.7mm_Pad, F.Cu at (68.6, 53.3)
- added REF**: MountingHole_3.7mm_Pad, MountingHole:MountingHole_3.7mm_Pad, F.Cu at (172.7, 53.3)
- added REF**: MountingHole_3.7mm_Pad, MountingHole:MountingHole_3.7mm_Pad, F.Cu at (68.6, 147.3)
- J10: renamed from ENC3; value Conn_01x04_Male -> ENC3
- J11: renamed from LoadCell1; value Conn_01x02_Male -> LoadCell1
- J12: renamed from LoadCell2; value Conn_01x02_Male -> LoadCell2
- J13: renamed from 5V1; value Conn_01x03_Male -> 5V1
- J7: value UWBchip -> GND1; footprint teensy:5pinJST -> teensy:4pinJST
- J8: renamed from ENC1; value Conn_01x04_Male -> ENC1
- J9: renamed from ENC2; value Conn_01x04_Male -> ENC2
- moved J1 132.3 mm to (131.0, 141.8)
- moved J6 127.3 mm to (151.4, 140.7), turned to 180 degrees
- moved LevelShifterUWB(5->3.3)1 127.1 mm to (145.3, 98.7), turned to 180 degrees
- moved J13 112.2 mm to (108.8, 60.8)
- moved J2 88.3 mm to (160.6, 116.3), turned to 90 degrees
- moved J3 88.3 mm to (160.7, 131.0), turned to 90 degrees
- moved J4 86.8 mm to (160.5, 101.1), turned to 90 degrees
- moved J7 74.7 mm to (138.8, 61.0), turned to 0 degrees
- moved R_PullDownUWB1 74.2 mm to (151.5, 92.7), turned to 180 degrees
- moved R1 67.1 mm to (101.0, 65.4), turned to 180 degrees
- moved C1 60.9 mm to (96.1, 78.3), turned to 180 degrees
- moved R2 57.4 mm to (101.0, 71.6), turned to 180 degrees
- moved R3 56.9 mm to (101.1, 95.6), turned to 180 degrees
- moved R6 55.6 mm to (102.6, 132.8), turned to 180 degrees
- moved R5 51.9 mm to (102.5, 126.4), turned to 180 degrees
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Connections:
- J7 pad 2: +3.3V -> GND
- J7 pad 3: /MOSI -> GND
- J7 pad 4: /MISO -> GND
Routing:
- net +3.3V: track 0.00 -> 249.8 mm, vias 0 -> 8
- net +5V: track 0.00 -> 192.7 mm
- net /TX: track 0.00 -> 88.1 mm
- net /RX: track 0.00 -> 68.7 mm
- net /Enc2B: track 0.00 -> 68.3 mm
- net GND: track 0.00 -> 57.6 mm
- net /TX1: track 0.00 -> 56.2 mm
- net /Enc2A: track 0.00 -> 51.8 mm
- net /B1: track 0.00 -> 50.0 mm
- net /B2: track 0.00 -> 47.2 mm
- net /B: track 0.00 -> 44.2 mm
- net /A: track 0.00 -> 43.2 mm
- net /Enc1B: track 0.00 -> 42.6 mm
- net /RX1: track 0.00 -> 41.2 mm
- net /EncA: track 0.00 -> 40.1 mm
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- added copper zone on B.Cu, net GND
Other:
- board outline added: 119.4 x 109.2 mm
