File: FinalTeensyBreakoutBoard/FinalTeensyBreakoutBoard.kicad_sch (KiCad schematic)
At the start: 36 parts, among them J1 POWER, J10 ENC3, J11 LoadCell1, J12 LoadCell2, J13 5V1, J2 MC1, J3 MC2, J4 MC3, J5 CurrSB, J6 UWB1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

Commit message: Add files via upload
Parts:
- R1, R2, R3, R4, R5, R6: footprint teensy:100ohmR -> teensy:100ohmRnew
Connections:
- net MISO: no longer names the net of U1.14 (12_MISO_MQSL)
- net MOSI: no longer names the net of U1.13 (11_MOSI_CTX1)
- net SCK: no longer names the net of U1.35 (13_SCK_LED)
- no-connect marks 43 -> 46
Changed lines of the file:
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@@
   (junction (at 106.68 55.88) (diameter 0) (color 0 0 0 0)
   )
+  (no_connect (at 238.76 91.44))
   (no_connect (at 179.07 111.76))
   (no_connect (at 179.07 114.3))
@@
   (no_connect (at 234.95 106.68))
   (no_connect (at 234.95 101.6))
+  (no_connect (at 175.26 91.44))
+  (no_connect (at 175.26 88.9))
   (no_connect (at 234.95 123.19))
   (no_connect (at 234.95 128.27))
@@
     (effects (font (size 1.27 1.27)) (justify left bottom))
   )
-  (label "MOSI" (at 175.26 88.9 180) (fields_autoplaced)
-    (effects (font (size 1.27 1.27)) (justify right bottom))
-  )
   (label "Enc1B" (at 158.75 73.66 0) (fields_autoplaced)
     (effects (font (size 1.27 1.27)) (justify left bottom))
@@
     (effects (font (size 1.27 1.27)) (justify left bottom))
   )
-  (label "MISO" (at 175.26 91.44 180) (fields_autoplaced)
-    (effects (font (size 1.27 1.27)) (justify right bottom))
-  )
   (label "SCL" (at 265.43 110.49 0) (fields_autoplaced)
     (effects (font (size 1.27 1.27)) (justify left bottom))
@@
   )
   (label "A2'" (at 101.6 160.02 0) (fields_autoplaced)
-    (effects (font (size 1.27 1.27)) (justify left bottom))
-  )
-  (label "SCK" (at 238.76 91.44 0) (fields_autoplaced)
     (effects (font (size 1.27 1.27)) (justify left bottom))
   )
@@
       (effects (font (size 1.27 1.27)) (justify left))
     )
-    (property "Footprint" "teensy:100ohmR" (at 94.996 156.464 90)
+    (property "Footprint" "teensy:100ohmRnew" (at 94.996 156.464 90)
       (effects (font (size 1.27 1.27)) hide)
     )
@@
       (effects (font (size 1.27 1.27)) (justify left))
     )
-    (property "Footprint" "teensy:100ohmR" (at 98.806 99.314 90)
+    (property "Footprint" "teensy:100ohmRnew" (at 98.806 99.314 90)
       (effects (font (size 1.27 1.27)) hide)
     )
@@
       (effects (font (size 1.27 1.27)) (justify left))
     )
-    (property "Footprint" "teensy:100ohmR" (at 97.536 68.834 90)
+    (property "Footprint" "teensy:100ohmRnew" (at 97.536 68.834 90)
       (effects (font (size 1.27 1.27)) hide)
     )
@@
       (effects (font (size 1.27 1.27)) (justify left))
     )
-    (property "Footprint" "teensy:100ohmR" (at 97.536 127.254 90)
+    (property "Footprint" "teensy:100ohmRnew" (at 97.536 127.254 90)
       (effects (font (size 1.27 1.27)) hide)
     )
@@
       (effects (font (size 1.27 1.27)) (justify left))
     )
-    (property "Footprint" "teensy:100ohmR" (at 93.726 183.134 90)
+    (property "Footprint" "teensy:100ohmRnew" (at 93.726 183.134 90)
       (effects (font (size 1.27 1.27)) hide)
     )
@@
       (effects (font (size 1.27 1.27)) (justify left))
     )
-    (property "Footprint" "teensy:100ohmR" (at 97.536 37.084 90)
-      (effects (font (size 1.27 1.27)) hide)
-    )
+    (property "Footprint" "teensy:100ohmRnew" (at 97.536 37.084 90)
+      (effects (font (size 1.27 1.27)) hide)
+    )
