File: FinalTeensyBreakoutBoard/_autosave-FinalTeensyBreakoutBoard.kicad_sch (KiCad schematic)
At the start: 38 parts, among them J1 POWER, J2 MC1, J3 MC2, J4 MC3, J5 CurrSB, J6 UWB1, J7 UWBchip, U1 Teensy4.1, U2 MAX3284E, U3 MAX3284E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

Commit message: finished layout
Parts:
- removed 3.3V1, GND1: Conn_01x03_Male, teensy:3pinJST, symbol Connector:Conn_01x03_Male
- removed J7: UWBchip, teensy:5pinJST, symbol Connector:Conn_01x05_Male
- added J7: GND1, teensy:4pinJST, symbol Connector:Conn_01x04_Pin
- J10: renamed from ENC3; value Conn_01x04_Male -> ENC3
- J11: renamed from LoadCell1; value Conn_01x02_Male -> LoadCell1
- J12: renamed from LoadCell2; value Conn_01x02_Male -> LoadCell2
- J13: renamed from 5V1; value Conn_01x03_Male -> 5V1
- J8: renamed from ENC1; value Conn_01x04_Male -> ENC1
- J9: renamed from ENC2; value Conn_01x04_Male -> ENC2
Connections:
- net GND: now also J7.1 (Pin_1), J7.2 (Pin_2), J7.3 (Pin_3), J7.4 (Pin_4)
